File: BladeCore-M40/src/HardwareDesign/BladeCore-M40.brd (EAGLE design)
At the start: 22 x 42 mm, 76 parts, among them IC1 CAT24C512HU5IGT3, IC2 PI3USB102J, IC3 W25Q128JVCIQ TR, IC4 RP-2040, IC5 MCP6001R, IC6 MIC5504-3.3YM5-TR, IC7 FT232RNQ, IC8 AP7335-WG-7, X1 12MHz

Commit message: Start with M54
Parts:
- renumbered R17 to J1, R18 to J2, R30 to J3
Changed lines of the file:
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@@
 <drawing>
 <settings>
-<setting alwaysvectorfont="yes"/>
+<setting alwaysvectorfont="no"/>
 <setting verticaltext="up"/>
 </settings>
@@
 <attribute name="VALUE" x="10.44" y="43.44" size="1.27" layer="27" ratio="10" rot="R180"/>
 </element>
-<element name="R30" library="ds_passive" package="R0201" package3d_urn="urn:adsk.eagle:package:47403529/3" value="DNI" x="10.52" y="27.76" smashed="yes" rot="R180">
+<element name="J3" library="ds_passive" package="R0201" package3d_urn="urn:adsk.eagle:package:47403529/3" value="DNI" x="10.52" y="27.76" smashed="yes" rot="R180">
 <attribute name="VALUE" x="11.155" y="29.665" size="1.016" layer="27" rot="R180"/>
 </element>
@@
 <attribute name="VALUE" x="16.735" y="13.535" size="1.27" layer="27" rot="R180"/>
 </element>
-<element name="R17" library="ds_passive" package="R0201" package3d_urn="urn:adsk.eagle:package:47403529/3" value="0R" x="8" y="39.91" smashed="yes" rot="MR0">
+<element name="J1" library="ds_passive" package="R0201" package3d_urn="urn:adsk.eagle:package:47403529/3" value="0R" x="8" y="39.91" smashed="yes" rot="MR0">
 <attribute name="VALUE" x="8.635" y="38.005" size="1.27" layer="28" rot="MR0"/>
 </element>
-<element name="R18" library="ds_passive" package="R0201" package3d_urn="urn:adsk.eagle:package:47403529/3" value="DNI" x="7.98" y="40.65" smashed="yes" rot="MR180">
+<element name="J2" library="ds_passive" package="R0201" package3d_urn="urn:adsk.eagle:package:47403529/3" value="DNI" x="7.98" y="40.65" smashed="yes" rot="MR180">
 <attribute name="VALUE" x="7.345" y="42.555" size="1.27" layer="28" rot="MR180"/>
 </element>
@@
 <wire x1="6.02" y1="7.38" x2="5.23" y2="6.59" width="0.508" layer="16"/>
 <wire x1="5.23" y1="6.59" x2="5.23" y2="2.91" width="0.508" layer="16"/>
-<contactref element="R18" pad="2"/>
+<contactref element="J2" pad="2"/>
 <wire x1="8.255" y1="40.65" x2="9.105" y2="41.5" width="0.1697" layer="16"/>
 <wire x1="9.105" y1="41.5" x2="10.1" y2="41.5" width="0.1697" layer="16"/>
@@
 <wire x1="6.13" y1="5.62739375" x2="5.645" y2="6.11239375" width="0.3048" layer="1"/>
 <wire x1="5.645" y1="6.11239375" x2="5.645" y2="6.325" width="0.3048" layer="1"/>
-<contactref element="R17" pad="1"/>
+<contactref element="J1" pad="1"/>
 <wire x1="4.57" y1="38.71" x2="4.57" y2="38.9528" width="0.1697" layer="16"/>
 <via x="4.57" y="38.9528" extent="1-16" drill="0.15"/>
@@
 <contactref element="C31" pad="1"/>
 <contactref element="C22" pad="1"/>
-<contactref element="R30" pad="2"/>
+<contactref element="J3" pad="2"/>
 <contactref element="C24" pad="1"/>
 <contactref element="IC4" pad="23"/>
@@
 </signal>
 <signal name="VREGO">
-<contactref element="R30" pad="1"/>
+<contactref element="J3" pad="1"/>
 <contactref element="IC4" pad="45"/>
 <contactref element="C23" pad="1"/>
@@
 <signal name="N$2">
 <contactref element="IC8" pad="3"/>
-<contactref element="R17" pad="2"/>
-<contactref element="R18" pad="1"/>
+<contactref element="J1" pad="2"/>
+<contactref element="J2" pad="1"/>
 <wire x1="7.705" y1="40.65" x2="7.725" y2="40.63" width="0.1697" layer="16"/>
 <wire x1="7.725" y1="40.63" x2="7.725" y2="39.91" width="0.1697" layer="16"/>
