File: BladeCore-M40/src/HardwareDesign/BladeCore-M40.sch (EAGLE design)
At the start: 76 parts, among them IC1 CAT24C512HU5IGT3, IC2 PI3USB102J, IC3 W25Q128JVPIQ, IC4 RP2040, IC5 MCP6001R, IC6 MIC5504-3.3YM5-TR, IC7 FT232RNQ, IC8 AP7335-WG-7, X1 12MHz

Commit message: Finish M40 design
Parts:
- removed BOOT, RUN: TPPAD1-13, testpad:TPPAD1-13
- removed R25, R26: 10K, ds_passive:R0201
- removed VCORE: TP, ds_passive:TP
- added R17, R3, R4: 0R, ds_passive:R0201
- added R18: DNI, ds_passive:R0201
- C21: value 100nF -> 4.7uF; device ds_passive:C-0201 -> ds_passive:C-0402
- IC3: value W25Q128JVPIQ -> W25Q128JVCIQ TR; device MCU:W25Q128JVP -> ds_ic_memory:W25Q128JVC
- IC4: value RP2040 -> RP-2040; device ds_ic_mcu:RP2040 -> ds_ic_mcu:RP-2040
- IC7: device ftdichip:FT232RQ -> ds_ic_peripherals:FT232RQ
- R11: value 1K -> 0R
- R23, R24: value 10K -> 3.3K
- R30: value 0R -> DNI
- RX: value CHIP-FLAT-G_0603-0.35MM -> CHIP-FLAT-G_0402; device LED:CHIP-FLAT-G_0603-0.35MM -> LED:CHIP-FLAT-G_0402
- TX: value CHIP-FLAT-B_0603-0.35MM -> CHIP-FLAT-B_0402; device LED:CHIP-FLAT-B_0603-0.35MM -> LED:CHIP-FLAT-B_0402
Connections:
- net N$1 renamed VFB
- net N$3 renamed FBTRIM
- net N$4 renamed FT_TX
- net N$5 renamed FT_RX
- removed net GP25/USBSEL: IC2.SEL, IC4.GPIO25, M.2-M1.39, R5.2, R7.1
- removed net I2C1_SCL: IC1.SCL, IC4.GPIO3, M.2-M1.4, R25.2
- removed net I2C1_SDA: IC1.SDA, IC4.GPIO2, M.2-M1.2, R26.2
- removed net N$7: IC4.VREG_VOUT, R30.1
- removed net SPI0_CS: IC4.GPIO17, M.2-M1.21
- removed net SPI0_MISO: IC4.GPIO16, M.2-M1.19
- removed net SPI0_MOSI: IC4.GPIO19, M.2-M1.25
- removed net SPI0_SCK: IC4.GPIO18, M.2-M1.23
- removed net SPI1_CS: IC4.GPIO13, M.2-M1.26
- removed net SPI1_MISO: IC4.GPIO12, M.2-M1.24
- removed net SPI1_MOSI: IC4.GPIO11, M.2-M1.22
- removed net SPI1_SCLK: IC4.GPIO10, M.2-M1.20
- removed net UART0_RX: IC4.GPIO1, R31.1
- removed net UART0_TX: IC4.GPIO0, R29.2
- removed net UART1_RX: IC4.GPIO9, M.2-M1.8, R12.2
- removed net UART1_TX: IC4.GPIO8, M.2-M1.10, R13.1
- removed net USB_BOOT: BOOT.TP, M.2-M1.48, R11.1
- new net DETECT: DETECT.C, M.2-M1.57
- new net GP0: IC4IO.GPIO0, M.2-M1.31, R29.2
- new net GP1: IC4IO.GPIO1, M.2-M1.29, R31.1
- new net GP10: IC4IO.GPIO10, M.2-M1.11
- new net GP11: IC4IO.GPIO11, M.2-M1.9
- new net GP12: IC4IO.GPIO12, M.2-M1.7
- new net GP13: IC4IO.GPIO13, M.2-M1.5
- new net GP16: IC4IO.GPIO16, M.2-M1.28
- new net GP17: IC4IO.GPIO17, M.2-M1.26
- new net GP18: IC4IO.GPIO18, M.2-M1.24
- new net GP19: IC4IO.GPIO19, M.2-M1.22
- new net GP2: IC4IO.GPIO2, M.2-M1.27
- new net GP25: IC4IO.GPIO25, M.2-M1.10, R11.2
- new net GP3: IC4IO.GPIO3, M.2-M1.25
- new net GP4: IC4IO.GPIO4, M.2-M1.23, R23.2, R4.1
- new net GP5: IC4IO.GPIO5, M.2-M1.21, R24.2, R3.1
- new net GP8: IC4IO.GPIO8, M.2-M1.15, R13.1
- new net GP9: IC4IO.GPIO9, M.2-M1.13, R12.2
- new net MUXSEL: IC2.SEL, R11.1, R5.2, R7.1
- new net VREGO: C23.1, IC4PWR.VREG_VOUT, R30.1
- net !QSPI_SS: now also IC4PWR.QSPI_SS_N; no longer IC4.QSPI_SS_N, R11.2
- net +3V3_MCU: now also IC4PWR.IOVDD1, IC4PWR.IOVDD2, IC4PWR.IOVDD3, IC4PWR.IOVDD4, IC4PWR.IOVDD5, IC4PWR.IOVDD6, IC4PWR.USB_VDD, IC4PWR.VREG_VIN, R17.1; no longer IC4.IOVDD, IC4.USB_VDD, IC4.VREG_VIN, IC8.EN, R25.1, R26.1
- net AD0: now also IC4IO.GPIO26, M.2-M1.8; no longer IC4.GPIO26/ADC0, M.2-M1.30
- net AD1: now also IC4IO.GPIO27, M.2-M1.6; no longer IC4.GPIO27/ADC1, M.2-M1.34
- net AD2: now also IC4IO.GPIO28, M.2-M1.4; no longer IC4.GPIO28/ADC2, M.2-M1.38
- net AD3: now also IC4IO.GPIO29, M.2-M1.2; no longer IC4.GPIO29/ADC3, M.2-M1.42
- net AVDD: now also IC4PWR.ADC_AVDD; no longer IC4.ADC_AVDD
- net GND: now also IC4PWR.GND, IC4PWR.TESTEN, M.2-M1.30, M.2-M1.33, M.2-M1.52, R18.2; no longer IC4.GND, IC4.TESTEN, M.2-M1.11, M.2-M1.12, M.2-M1.17, M.2-M1.18, M.2-M1.27, M.2-M1.28, M.2-M1.36, M.2-M1.40, M.2-M1.41, M.2-M1.44, M.2-M1.5, M.2-M1.50, M.2-M1.56, M.2-M1.57, M.2-M1.6, M.2-M1.7, M.2-M1.9
- net GP14: now also IC4IO.GPIO14, M.2-M1.3; no longer IC4.GPIO14, M.2-M1.16
- net GP15: now also IC4IO.GPIO15, M.2-M1.1; no longer IC4.GPIO15, M.2-M1.14
- net GP20: now also IC4IO.GPIO20, M.2-M1.20; no longer IC4.GPIO20, M.2-M1.29
- net GP21: now also IC4IO.GPIO21, M.2-M1.18; no longer IC4.GPIO21, M.2-M1.31
- net GP22: now also IC4IO.GPIO22, M.2-M1.16; no longer IC4.GPIO22, M.2-M1.33
- net GP23: now also IC4IO.GPIO23, M.2-M1.14; no longer IC4.GPIO23, M.2-M1.35
- net GP24: now also IC4IO.GPIO24, M.2-M1.12; no longer IC4.GPIO24, M.2-M1.37
- net GP6: now also IC4IO.GPIO6, M.2-M1.19; no longer IC4.GPIO6, M.2-M1.13
- net GP7: now also IC4IO.GPIO7, M.2-M1.17; no longer IC4.GPIO7, M.2-M1.15
- net I2C0_SCL: now also IC1.SCL, R3.2; no longer IC4.GPIO5, M.2-M1.3, R23.2
- net I2C0_SDA: now also IC1.SDA, R4.2; no longer IC4.GPIO4, M.2-M1.1, R24.2
- net N$2: now also IC8.EN, R17.2, R18.1; no longer DETECT.C, M.2-M1.58
- net QSPI_SCLK: now also IC4PWR.QSPI_SCLK; no longer IC4.QSPI_SCLK
- net QSPI_SD0: now also IC4PWR.QSPI_SD0; no longer IC4.QSPI_SD0
- net QSPI_SD1: now also IC4PWR.QSPI_SD1; no longer IC4.QSPI_SD1
- net QSPI_SD2: now also IC4PWR.QSPI_SD2; no longer IC4.QSPI_SD2
- net QSPI_SD3: now also IC4PWR.QSPI_SD3; no longer IC4.QSPI_SD3
- net RP_XI: now also IC4PWR.XIN; no longer IC4.XIN
- net RP_XO: now also IC4PWR.XOUT; no longer IC4.XOUT
- net RUN: now also IC4PWR.RUN, M.2-M1.54; no longer IC4.RUN, M.2-M1.46, RUN.TP
- net SWCLK: now also IC4PWR.SWCLK; no longer IC4.SWCLK
- net SWCLK_M2: now also M.2-M1.58; no longer M.2-M1.43
- net SWDIO: now also IC4PWR.SWDIO; no longer IC4.SWDIO
- net SWDIO_M2: now also M.2-M1.56; no longer M.2-M1.45
- net USBRP2_DP_N: now also IC4PWR.USB_DM; no longer IC4.USB_DM
- net USBRP2_DP_P: now also IC4PWR.USB_DP; no longer IC4.USB_DP
- net VCORE: now also IC4PWR.DVDD1, IC4PWR.DVDD2; no longer C23.1, IC4.DVDD, VCORE.P$1
Other:
- moved on the sheet: C1, C10, C11, C12, C13, C14, C15, C16, C17, C18, C19, C2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

Commit message: Start with M54
Parts:
- renumbered R17 to J1, R18 to J2, R30 to J3
Changed lines of the file:
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@@
 <part name="R1" library="Resistor_Capacitor" library_urn="urn:adsk.eagle:library:15122775" deviceset="35WR10KLFTR" device="" package3d_urn="urn:adsk.eagle:package:10872895/3" value="25K"/>
 <part name="GND2" library="ds_passive" deviceset="GND" device=""/>
-<part name="R30" library="ds_passive" deviceset="R" device="0201" package3d_urn="urn:adsk.eagle:package:47403529/3" value="DNI"/>
+<part name="J3" library="ds_passive" deviceset="R" device="0201" package3d_urn="urn:adsk.eagle:package:47403529/3" value="DNI"/>
 <part name="C30" library="ds_passive" deviceset="C" device="-0402" package3d_urn="urn:adsk.eagle:package:46766485/2" value="4.7uF"/>
 <part name="C9" library="ds_passive" deviceset="C" device="-0201" package3d_urn="urn:adsk.eagle:package:47403530/3" value="100nF"/>
@@
 <part name="NC27" library="ds_passive" deviceset="NC" device=""/>
 <part name="R11" library="ds_passive" deviceset="R" device="0201" package3d_urn="urn:adsk.eagle:package:47403529/3" value="0R"/>
-<part name="R17" library="ds_passive" deviceset="R" device="0201" package3d_urn="urn:adsk.eagle:package:47403529/3" value="0R"/>
-<part name="R18" library="ds_passive" deviceset="R" device="0201" package3d_urn="urn:adsk.eagle:package:47403529/3" value="DNI"/>
+<part name="J1" library="ds_passive" deviceset="R" device="0201" package3d_urn="urn:adsk.eagle:package:47403529/3" value="0R"/>
+<part name="J2" library="ds_passive" deviceset="R" device="0201" package3d_urn="urn:adsk.eagle:package:47403529/3" value="DNI"/>
 </parts>
 <sheets>
@@
 <attribute name="VALUE" x="728.98" y="96.52" size="1.778" layer="96" align="top-center"/>
 </instance>
-<instance part="R30" gate="G$1" x="439.42" y="254" smashed="yes" rot="R270">
+<instance part="J3" gate="G$1" x="439.42" y="254" smashed="yes" rot="R270">
 <attribute name="NAME" x="436.245" y="255.4986" size="1.778" layer="95"/>
 <attribute name="VALUE" x="438.785" y="250.698" size="1.778" layer="96"/>
@@
 <attribute name="VALUE" x="460.375" y="191.008" size="1.778" layer="96"/>
 </instance>
-<instance part="R17" gate="G$1" x="665.48" y="132.08" smashed="yes" rot="MR0">
+<instance part="J1" gate="G$1" x="665.48" y="132.08" smashed="yes" rot="MR0">
 <attribute name="NAME" x="666.9786" y="128.905" size="1.778" layer="95" rot="MR90"/>
 <attribute name="VALUE" x="662.178" y="131.445" size="1.778" layer="96" rot="MR90"/>
 </instance>
-<instance part="R18" gate="G$1" x="665.48" y="116.84" smashed="yes" rot="MR0">
+<instance part="J2" gate="G$1" x="665.48" y="116.84" smashed="yes" rot="MR0">
 <attribute name="NAME" x="666.9786" y="113.665" size="1.778" layer="95" rot="MR90"/>
 <attribute name="VALUE" x="662.178" y="116.205" size="1.778" layer="96" rot="MR90"/>
@@
 <wire x1="678.18" y1="132.08" x2="675.64" y2="132.08" width="0.1524" layer="91"/>
 <wire x1="675.64" y1="132.08" x2="675.64" y2="109.22" width="0.1524" layer="91"/>
-<pinref part="R18" gate="G$1" pin="2"/>
+<pinref part="J2" gate="G$1" pin="2"/>
 <wire x1="675.64" y1="109.22" x2="675.64" y2="101.6" width="0.1524" layer="91"/>
 <wire x1="665.48" y1="111.76" x2="665.48" y2="109.22" width="0.1524" layer="91"/>
@@
 <wire x1="657.86" y1="132.08" x2="657.86" y2="139.7" width="0.1524" layer="91"/>
 <junction x="657.86" y="139.7"/>
-<pinref part="R17" gate="G$1" pin="1"/>
+<pinref part="J1" gate="G$1" pin="1"/>
 <wire x1="665.48" y1="137.16" x2="665.48" y2="139.7" width="0.1524" layer="91"/>
 <junction x="665.48" y="139.7"/>
@@
 </segment>
 <segment>
-<pinref part="R30" gate="G$1" pin="2"/>
+<pinref part="J3" gate="G$1" pin="2"/>
 <wire x1="434.34" y1="254" x2="391.16" y2="254" width="0.1524" layer="91"/>
 <label x="391.16" y="254" size="1.27" layer="95" rot="R180" xref="yes"/>
@@
 <net name="VREGO" class="0">
 <segment>
-<pinref part="R30" gate="G$1" pin="1"/>
+<pinref part="J3" gate="G$1" pin="1"/>
 <wire x1="444.5" y1="254" x2="449.58" y2="254" width="0.1524" layer="91"/>
 <label x="472.44" y="256.54" size="1.778" layer="95" rot="R180"/>
@@
 <wire x1="678.18" y1="137.16" x2="670.56" y2="137.16" width="0.1524" layer="91"/>
 <wire x1="670.56" y1="137.16" x2="670.56" y2="124.46" width="0.1524" layer="91"/>
-<pinref part="R17" gate="G$1" pin="2"/>
-<pinref part="R18" gate="G$1" pin="1"/>
+<pinref part="J1" gate="G$1" pin="2"/>
+<pinref part="J2" gate="G$1" pin="1"/>
 <wire x1="665.48" y1="121.92" x2="665.48" y2="124.46" width="0.1524" layer="91"/>
 <wire x1="665.48" y1="124.46" x2="665.48" y2="127" width="0.1524" layer="91"/>
