File: BladeCore-M54/src/HardwareDesign/BladeCore-M54.sch (EAGLE design)
At the start: 0 parts

Commit message: Start with M54
Parts:
- added C1, C2: 10uF, ds_passive:C0805
- added C10, C11, C33: 4.7uF, ds_passive:C-0201
- added C12, C13, C14, C15, C16, C17, C18, C22, C23, C24, C25, C26, C32, C34, C35, C36, C7: 100nF, ds_passive:C-0201
- added C21: 4.7uF, ds_passive:C-0402
- added C28, C29: 15pF, ds_passive:C-0201
- added C3, C4, C5: 100nF/16V, ds_passive:C-0201
- added C6: 4.7uF/16V, ds_passive:C-0201
- added DETECT, RX: CHIP-FLAT-G_0402, LED:CHIP-FLAT-G_0402
- added IC1: CAT24C512HU5IGT3, ds_ic_memory:CAT24C256-HU4
- added IC2: PI3USB102J, ds_ic_peripherals:PI3USB102JXUCEX
- added IC3: W25Q128JVCIQ TR, ds_ic_memory:W25Q128JVC
- added IC6: MIC5504-3.3YM5-TR, ds_ic_vreg:MIC5504-3.3YM5-TR
- added IC7: FT232RNQ, ds_ic_peripherals:FT232RQ
- added IC9: RP235XB, ds_ic_mcu:RP235XB
- added J3, R12, R13, R14, R7: DNI, ds_passive:R0201
- added L1: 3.3uH, ds_passive:L
- added M.2-M1: (no value), ds_con:M.2-M-KEY
- added R10, R16, R6, R9: 1K, ds_passive:R0201
- added R11, R15, R21, R22, R29, R3, R31, R4: 0R, ds_passive:R0201
- added R2: 33R, ds_passive:R0201
- added R23, R24: 3.3K, ds_passive:R0201
- added R32, R33: 22R, ds_passive:R0201
- added R5, R8: 10K, ds_passive:R0201
- added TX: CHIP-FLAT-B_0402, LED:CHIP-FLAT-B_0402
- added X1: 12MHz, Wurth_Quartz Crystals & Oscillators_WE-XTAL:WE-XTAL_CFPX-180_830069944
Connections:
- new net !QSPI_SS: IC3.!CS, IC9PWR.QSPI_SS
- new net +3V3_MCU: C12.1, C13.1, C14.1, C15.1, C16.1, C17.1, C18.1, C2.1, C21.1, C23.1, C26.1, C32.1, C34.1, C35.1, C36.1, C5.1, C7.1, IC1.VCC, IC2.VCC, IC3.VCC, IC6.VOUT, IC9PWR.ADC_AVDD, IC9PWR.IOVDD1, IC9PWR.IOVDD2, IC9PWR.IOVDD3, IC9PWR.IOVDD4, IC9PWR.IOVDD5, IC9PWR.IOVDD6, IC9PWR.IOVDD7, IC9PWR.IOVDD8, IC9PWR.QSPI_IOVDD, IC9PWR.USB_OTP_VDD, IC9PWR.VREG_IN, M.2-M1.67, M.2-M1.68, M.2-M1.69, R16.2, R2.1, R23.1, R24.1, R7.2, R8.1
- new net DETECT: DETECT.C, M.2-M1.57
- new net FT_RX: IC7.RXD, R13.2, R29.1
- new net FT_TX: IC7.TXD, R12.1, R31.2
- new net GND: C1.2, C10.2, C11.2, C12.2, C13.2, C14.2, C15.2, C16.2, C17.2, C18.2, C2.2, C21.2, C22.2, C23.2, C24.2, C25.2, C26.2, C28.2, C29.2, C3.2, C32.2, C33.2, C34.2, C35.2, C36.2, C4.2, C5.2, C6.2, C7.2, IC1.A0, IC1.A1, IC1.A2, IC1.GND, IC1.WP, IC2.!OE, IC2.GND, IC3.GND, IC6.GND, IC7.GND, IC7.GND@1, IC7.GND@2, IC7.GND@A, IC7.PAD, IC7.TEST, IC9PWR.GND, IC9PWR.VREG_PGND, M.2-M1.30, M.2-M1.33, M.2-M1.51, M.2-M1.52, M.2-M1.70, M.2-M1.71, M.2-M1.72, M.2-M1.MP1, R5.1, X1.GND
- new net GP0: IC9GPIO1.GPIO0, M.2-M1.31, R29.2
- new net GP1: IC9GPIO1.GPIO1, M.2-M1.29, R31.1
- new net GP10: IC9GPIO1.GPIO10, M.2-M1.11
- new net GP11: IC9GPIO1.GPIO11, M.2-M1.9
- new net GP12: IC9GPIO1.GPIO12, M.2-M1.7
- new net GP13: IC9GPIO1.GPIO13, M.2-M1.5
- new net GP14: IC9GPIO1.GPIO14, M.2-M1.3
- new net GP15: IC9GPIO1.GPIO15, M.2-M1.1
- new net GP16: IC9GPIO1.GPIO16, M.2-M1.28
- new net GP17: IC9GPIO1.GPIO17, M.2-M1.26
- new net GP18: IC9GPIO1.GPIO18, M.2-M1.24
- new net GP19: IC9GPIO1.GPIO19, M.2-M1.22
- new net GP2: IC9GPIO1.GPIO2, M.2-M1.27
- new net GP20: IC9GPIO1.GPIO20, M.2-M1.20
- new net GP21: IC9GPIO1.GPIO21, M.2-M1.18
- new net GP22: IC9GPIO1.GPIO22, M.2-M1.16
- new net GP23: IC9GPIO1.GPIO23, M.2-M1.14
- new net GP24: IC9GPIO1.GPIO24, M.2-M1.12
- new net GP25: IC9GPIO1.GPIO25, M.2-M1.10, R11.2
- new net GP26: IC9GPIO1.GPIO26, M.2-M1.8
- new net GP27: IC9GPIO1.GPIO27, M.2-M1.6
- new net GP28: IC9GPIO1.GPIO28, M.2-M1.4
- new net GP29: IC9GPIO1.GPIO29, M.2-M1.2
- new net GP3: IC9GPIO1.GPIO3, M.2-M1.25
- new net GP30: IC9GPIO2.GPIO30, M.2-M1.32
- new net GP31: IC9GPIO2.GPIO31, M.2-M1.34
- new net GP32: IC9GPIO2.GPIO32, M.2-M1.36
- new net GP33: IC9GPIO2.GPIO33, M.2-M1.38
- new net GP34: IC9GPIO2.GPIO34, M.2-M1.40
- new net GP35: IC9GPIO2.GPIO35, M.2-M1.42
- new net GP36: IC9GPIO2.GPIO36, M.2-M1.44
- new net GP37: IC9GPIO2.GPIO37, M.2-M1.46
- new net GP38: IC9GPIO2.GPIO38, M.2-M1.48
- new net GP39: IC9GPIO2.GPIO39, M.2-M1.50
- new net GP4: IC9GPIO1.GPIO4, M.2-M1.23, R23.2, R4.1
- new net GP40: IC9GPIO2.GPIO40_ADC0, M.2-M1.49
- new net GP41: IC9GPIO2.GPIO41_ADC1, M.2-M1.47
- new net GP42: IC9GPIO2.GPIO42_ADC2, M.2-M1.45
- new net GP43: IC9GPIO2.GPIO43_ADC3, M.2-M1.43
- new net GP44: IC9GPIO2.GPIO44_ADC4, M.2-M1.41
- new net GP45: IC9GPIO2.GPIO45_ADC5, M.2-M1.39
- new net GP46: IC9GPIO2.GPIO46_ADC6, M.2-M1.37
- new net GP47: IC9GPIO2.GPIO47_ADC7, M.2-M1.35
- new net GP5: IC9GPIO1.GPIO5, M.2-M1.21, R24.2, R3.1
- new net GP6: IC9GPIO1.GPIO6, M.2-M1.19
- new net GP7: IC9GPIO1.GPIO7, M.2-M1.17
- new net GP8: IC9GPIO1.GPIO8, M.2-M1.15, R13.1
- new net GP9: IC9GPIO1.GPIO9, M.2-M1.13, R12.2
- new net I2C0_SCL: IC1.SCL, R3.2
- new net I2C0_SDA: IC1.SDA, R4.2
- new net LX: IC9PWR.VREG_LX, L1.2
- new net MUXSEL: IC2.SEL, R11.1, R5.2, R7.1
- new net N$109: IC7.CBUS1, R9.1
- new net N$110: R9.2, TX.C
- new net N$111: R10.2, RX.C
- new net N$43: IC7.CBUS0, R10.1
- new net N$53: C29.1, R6.1, X1.1
- new net N$6: DETECT.A, R16.1
- new net QSPI_SCLK: IC3.CLK, IC9PWR.QSPI_SCLK
- new net QSPI_SD0: IC3.DI/IO0, IC9PWR.QSPI_SD0
- new net QSPI_SD1: IC3.DO/IO1, IC9PWR.QSPI_SD1
- new net QSPI_SD2: IC3.!WP!/IO2, IC9PWR.QSPI_SD2
- new net QSPI_SD3: IC3.!HOLD!/IO3, IC9PWR.QSPI_SD3
- new net REGO: C4.1, IC7.3V3OUT, R15.1
- new net RP_XI: C28.1, IC9PWR.XIN, X1.2
- new net RP_XO: IC9PWR.XOUT, R6.2
- new net RUN: IC9PWR.RUN, M.2-M1.54, R8.2
- new net SWCLK: IC9PWR.SWCLK, R22.2
- new net SWCLK_M2: M.2-M1.58, R22.1
- new net SWDIO: IC9PWR.SWDIO, R21.2
- new net SWDIO_M2: M.2-M1.56, R21.1
- new net USBFT_DP_N: IC2.D-, IC7.USBDM
- new net USBFT_DP_P: IC2.D+, IC7.USBDP
- new net USBRP2_DP_N: IC9PWR.USB_DM, R32.2
- new net USBRP2_DP_P: IC9PWR.USB_DP, R33.2
- new net USBRP_DP_N: IC2.M-, R32.1
- new net USBRP_DP_P: IC2.M+, R33.1
- new net USB_DP_N: IC2.Y-, M.2-M1.53
- new net USB_DP_P: IC2.Y+, M.2-M1.55
- new net VBUS: C1.1, C25.1, IC6.EN, IC6.VIN, IC7.VCC, M.2-M1.73, M.2-M1.74, M.2-M1.75, R14.2, RX.A, TX.A
- new net VCCIO: C3.1, C6.1, IC7.VCCIO, R14.1, R15.2
- new net VCORE: C10.1, C22.1, C24.1, IC9PWR.DVDD1, IC9PWR.DVDD2, IC9PWR.DVDD3, J3.2
- new net VREGO: C11.1, IC9PWR.VREG_FB, J3.1, L1.1
- new net VREG_AVDD: C33.1, IC9PWR.VREG_AVDD, R2.2
Other:
- note added: "1.0.0"
- note added: "3.3 VBUS-LDO"
- note added: "3.3V/5V select"
- note added: "BLADECORE-M40"
- note added: "David Sipos / DvidMakesThings"
- note added: "FLASH"
- note added: "M.2 CONNECTOR M-KEY"
- note added: "RP2354B MCU"
- note added: "USB MULTIPLEXER"
- note added: "USB-UART CONVERTER"
- note added: "USER MEMORY"
